File: sch/FA1/FA1.sch (KiCad schematic (older format))
At the start: 13 parts, among them J1 DMX OUT, J2 module_connector, U1 SP485E

Commit message: Renamed folders/files as per new coding convention (see README). Added FA1 and FA2 schematics. Updated all schematic title blocks.
Parts:
- removed C1: 10uF 10V, Resistor_SMD:R_0805_2012Metric, symbol Device:C
- removed C2: 100nF 50V, Resistor_SMD:R_0805_2012Metric, symbol Device:C
- removed D1, D2: 43V 600W, project_parts:D_SMB_NP, symbol Device:D_TVS_ALT
- removed J2: module_connector, project_parts:Light_controller_module, symbol light_controller:module_connector
- removed R1, R5, R6: 10k, Resistor_SMD:R_0805_2012Metric, symbol Device:R
- removed R2, R4: 10R, Resistor_SMD:R_0805_2012Metric, symbol Device:R
- removed R3: 120R, Resistor_SMD:R_0805_2012Metric, symbol Device:R
- removed U1: SP485E, project_parts:SOIC-8_3.9x4.9mm_P1.27mm, symbol Interface_UART:MAX485E
- added J2: Cellular Antenna, symbol Connector:Conn_Coaxial
- added J3: DMX Out, symbol Connector_Generic:Conn_01x04
- added U1: FP1 sub-assembly, symbol faraday:FP1
- added U2: PS-05-5, symbol faraday:PS-05
- J1: value DMX OUT -> 240V mains; footprint TerminalBlock_Phoenix:TerminalBlock_Phoenix_MKDS-1,5-3-5.08_1x03_P5.08mm_Horizontal -> (none); Description (none) -> PWR ENT RCPT IEC320-C14 PANEL QC; Manufacturer On Shore Technology -> Qualtek; Order Number ED2903-ND -> Q212-ND; Part Number OSTYC032150 -> 703W-00/04
Connections:
- net labels added: Earth
- net labels removed: +5V, RS485_DRV_EN, RS485_RCV_EN, UART_RX, UART_TX
- wire segments 56 -> 31
- no-connect marks 10 -> 0
Other:
- note added: "Optional"
- note removed: "DMX Output (RS485)"
- note removed: "To motherboard"
