File: sch/FP1/FP1.sch (KiCad schematic (older format))
At the start: 63 parts, among them J1 240V Mains, J2 Module 0, J3 5VDC, J4 Module 1, J5 Power LED, J6 Connection LED, U1 Electron

Commit message: Renamed folders/files as per new coding convention (see README). Added FA1 and FA2 schematics. Updated all schematic title blocks.
Parts:
- J2, J4: footprint project_parts:Light_controller_module -> project_parts:Faraday_module; symbol light_controller:module_connector -> faraday:module_connector
- PS1: symbol light_controller:LHE15-20Dxx -> faraday:LHE15-20Dxx
- U1: symbol light_controller:PARTICLE_ELECTRON -> faraday:PARTICLE_ELECTRON
Other:
- moved on the sheet: C6, C7, J3, R1, R2
